File: PCB/MidiControllerPCB.kicad_pcb (KiCad board)
At the start: 2 copper layers, 215 x 139 mm, 1506 parts, among them J1 BARREL_JACK, J10 L10_Out, J11 L9_In, J12 L9_Out, J13 4_In, J14 4_Out, J15 3_In, J16 3_Out, J17 2_In, J18 2_Out, J19 1_In, J2 LMain_Out, J20 1_Out, J21 DIN_5, J22 Vol_In, J23 Vol_Out, J24 Tap1, J25 Tap2, J26 ToMainOutL, J27 MainOutL, J28 ToVolInOut, J29 VolInOut, J3 Tap3, J35 Raspberry_Pi_2_3, J4 Tap4, J41 PIC_debug, J44 pi 1=pwr 2=gnd, J5 LEDs / LCD / FootSwitches, J6 Pedal Routes, J7 DIN_5, J8 DIN_5, J9 L10_In, K1 AZ850-x, K10 AZ850-x, K11 AZ850-x, K12 AZ850-x, K13 AZ850-x, K14 AZ850-x, K15 AZ850-x, K16 AZ850-x, K17 AZ850-x, K2 AZ850-x, K3 AZ850-x, K4 AZ850-x, K5 AZ850-x, K6 AZ850-x, K7 AZ850-x, K8 AZ850-x, K9 AZ850-x, Q1 Q_NPN_BEC, Q10 Q_NPN_BEC, Q11 Q_NPN_BEC, Q12 Q_NPN_BEC, Q13 Q_NPN_BEC, Q14 Q_NPN_BEC, Q15 Q_NPN_BEC, Q16 Q_NPN_BEC, Q17 Q_NPN_BEC, Q18 Q_NPN_BEC, Q19 Q_NPN_BEC, Q2 Q_NPN_BEC, Q20 Q_NPN_BEC, Q21 Q_NPN_BEC, Q22 Q_NPN_BEC, Q3 Q_NPN_BEC, Q4 Q_NPN_BEC, Q5 Q_NPN_BEC, Q6 Q_NPN_BEC, Q7 Q_NPN_BEC, Q8 Q_NPN_BEC, Q9 Q_NPN_BEC, U1 MCP23017_ML, U10 PIC18F26K80_IML, U2 MCP23017_ML, U3 MCP23017_ML, U4 MCP23017_ML, U5 CD4050BCN, U6 4N35, U7 7805_PINS, U8 TL072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

Commit message: schematic: nothing todo list: modify notes
Parts:
- removed C15, C17: 10uf, Capacitors_THT:CP_Radial_D4.0mm_P2.00mm
- removed C16, C18: 0.1uf, Capacitors_THT:C_Axial_L3.8mm_D2.6mm_P7.50mm_Horizontal
- removed D1, D10, D11, D12, D13, D14, D15, D17, D2, D20, D22, D3, D4, D5, D6, D7, D8, D9: 1N4001, Diodes_SMD:D_SMA
- removed J10: L10_Out, NRJ6HM:NRJ6HM-1-PRE
- removed J11: L9_In, NRJ6HM:NRJ6HM-1-PRE
- removed J12: L9_Out, NRJ6HM:NRJ6HM-1-PRE
- removed J13: 4_In, NRJ6HM:NRJ6HM-1-PRE
- removed J14: 4_Out, NRJ6HM:NRJ6HM-1-PRE
- removed J15: 3_In, NRJ6HM:NRJ6HM-1-PRE
- removed J16: 3_Out, NRJ6HM:NRJ6HM-1-PRE
- removed J17: 2_In, NRJ6HM:NRJ6HM-1-PRE
- removed J18: 2_Out, NRJ6HM:NRJ6HM-1-PRE
- removed J19: 1_In, NRJ6HM:NRJ6HM-1-PRE
- removed J20: 1_Out, NRJ6HM:NRJ6HM-1-PRE
- removed J21: DIN_5, stomp:Midi-Connector
- removed J22: Vol_In, NRJ6HM:NRJ6HM-1-PRE
- removed J23: Vol_Out, NRJ6HM:NRJ6HM-1-PRE
- removed J26: ToMainOutL, Pin_Headers:Pin_Header_Straight_2x05_Pitch2.54mm
- removed J27: MainOutL, Pin_Headers:Pin_Header_Straight_2x05_Pitch2.54mm
- removed J28: ToVolInOut, Pin_Headers:Pin_Header_Straight_2x05_Pitch2.54mm
- removed J29: VolInOut, Pin_Headers:Pin_Header_Straight_2x05_Pitch2.54mm
- removed J44: pi 1=pwr 2=gnd, Pin_Headers:Pin_Header_Straight_1x02_Pitch2.54mm
- removed J5: LEDs / LCD / FootSwitches, Pin_Headers:Pin_Header_Straight_2x20_Pitch2.54mm
- removed J6: Pedal Routes, Pin_Headers:Pin_Header_Straight_2x20_Pitch2.54mm
- removed J9: L10_In, NRJ6HM:NRJ6HM-1-PRE
- removed K1, K10, K11, K12, K13, K14, K15, K16, K17, K2, K3, K4, K5, K6, K7, K8, K9: AZ850-x, Relays_THT:Relay_DPDT_FRT5
- removed Q1, Q10, Q11, Q12, Q13, Q14, Q15, Q16, Q17, Q18, Q19, Q2, Q20, Q21, Q22, Q3, Q4, Q5, Q6, Q7, Q8, Q9: Q_NPN_BEC, TO_SOT_Packages_SMD:SOT-23
- removed R34, R45: 100, Resistors_SMD:R_1206_HandSoldering
- removed R43: 1k, Resistors_SMD:R_1206_HandSoldering
- removed R57, R59, R61, R64: 470, Resistors_SMD:R_1206_HandSoldering
- removed R58, R60, R62, R65: 4.7k, Resistors_SMD:R_1206_HandSoldering
- removed R75, R76, R77, R78, R79: 2.2M, Resistors_SMD:R_0603_HandSoldering
- removed REF** (x1354): via, stomp:via
- removed REF** (x4): , Mounting_Holes:MountingHole_2.7mm
- removed TP1: 9V, Pin_Headers:Pin_Header_Straight_1x01_Pitch2.54mm
- removed TP2: GND, Pin_Headers:Pin_Header_Straight_1x01_Pitch2.54mm
- removed U1, U3, U4: MCP23017_ML, Housings_DFN_QFN:QFN-28-1EP_6x6mm_Pitch0.65mm
- removed U6: 4N35, Housings_DIP:DIP-6_W7.62mm_Socket
- removed U7: 7805_PINS, TO_SOT_Packages_THT:TO-220-3_Vertical
- removed U8, U9: TL072, Housings_SSOP:TSSOP-8_4.4x3mm_Pitch0.65mm
- added C1: 0.1uf, Capacitors_SMD:C_1206_HandSoldering, F.Cu at (166.1, 80.3)
- added C2: 0.1uf, Capacitors_SMD:C_1206_HandSoldering, F.Cu at (185.7, 103.2)
- added C3: 0.1uf, Capacitors_SMD:C_1206_HandSoldering, F.Cu at (178.1, 103.2)
- added C4: 0.1uf, Capacitors_SMD:C_1206_HandSoldering, F.Cu at (165.4, 56.0)
- added C5: 0.1uf, Capacitors_SMD:C_1206_HandSoldering, F.Cu at (166.1, 77.1)
- added C6: 0.01uf, Capacitors_SMD:C_1206_HandSoldering, F.Cu at (180.5, 56.0)
- added C7: 0.01uf, Capacitors_SMD:C_1206_HandSoldering, F.Cu at (173.0, 56.0)
- added R21: 10k, Resistors_SMD:R_1206_HandSoldering, F.Cu at (166.8, 66.9)
- added R22: 10k, Resistors_SMD:R_1206_HandSoldering, F.Cu at (181.2, 82.0)
- added R23: 1k, Resistors_SMD:R_1206_HandSoldering, F.Cu at (190.8, 71.4)
- added R24: 1k, Resistors_SMD:R_1206_HandSoldering, F.Cu at (190.8, 74.7)
- added R25: 10k, Resistors_SMD:R_1206_HandSoldering, F.Cu at (185.3, 100.0)
- added R26: 1k, Resistors_SMD:R_1206_HandSoldering, F.Cu at (175.1, 85.2)
- added R27: 10k, Resistors_SMD:R_1206_HandSoldering, F.Cu at (175.1, 88.5)
- added R28: 10k, Resistors_SMD:R_1206_HandSoldering, F.Cu at (184.4, 93.5)
- added R29: 10k, Resistors_SMD:R_1206_HandSoldering, F.Cu at (167.5, 86.8)
- added SW1: SW_SPST, Pin_Headers:Pin_Header_Straight_1x02_Pitch2.54mm, F.Cu at (168.3, 174.5)
- added SW2: SW_SPST, Pin_Headers:Pin_Header_Straight_1x02_Pitch2.54mm, F.Cu at (156.7, 173.7)
- added SW3: SW_SPST, Pin_Headers:Pin_Header_Straight_1x02_Pitch2.54mm, F.Cu at (96.5, 171.3)
- added SW4: SW_SPST, Pin_Headers:Pin_Header_Straight_1x02_Pitch2.54mm, F.Cu at (106.9, 172.6)
- added SW5: SW_SPST, Pin_Headers:Pin_Header_Straight_1x02_Pitch2.54mm, F.Cu at (143.8, 175.1)
- added SW6: RGB_Rotary_Enc_PB, Pin_Headers:Pin_Header_Straight_2x04_Pitch2.54mm, F.Cu at (69.6, 25.9)
- C13, C14: footprint Capacitors_THT:C_Axial_L3.8mm_D2.6mm_P7.50mm_Horizontal -> Capacitors_SMD:C_1206_HandSoldering
- J1: value BARREL_JACK -> OLED_Display; footprint Connectors:BARREL_JACK -> Pin_Headers:Pin_Header_Straight_1x07_Pitch1.00mm
- J2: value LMain_Out -> fan_header; footprint NRJ6HM:NRJ6HM-1-PRE -> Pin_Headers:Pin_Header_Straight_1x02_Pitch2.54mm
- J24: value Tap1 -> TRS_Midi_1
- J25: value Tap2 -> TRS_Midi_2
- J3: value Tap3 -> TRS_Midi_3
- J4: value Tap4 -> TRS_Midi_4
- J41, U2: moved to F.Cu
- R1, R2, R3, R4, R5, R6, R7, R8: value 100 -> 220
- R10, R11, R12, R13, R14, R30, R9: value 100 -> 10k
- R19: value 470 -> 10k
- R20: value 270 -> 10k
- moved J2 198.5 mm to (41.3, 107.4)
- moved J3 192.8 mm to (55.2, 163.8)
- moved J7 185.7 mm to (67.1, 80.9), turned to 0 degrees
- moved J4 182.5 mm to (56.3, 122.9)
- moved J8 175.6 mm to (68.2, 57.9), turned to 0 degrees
- moved R20 130.4 mm to (166.8, 63.6), turned to 0 degrees
- moved R74 119.1 mm to (182.6, 88.5), turned to 0 degrees
- moved R73 118.1 mm to (182.6, 85.2), turned to 0 degrees
- moved R19 111.4 mm to (184.4, 96.7), turned to 0 degrees
- moved R69 107.9 mm to (174.7, 67.6), turned to 0 degrees
- moved J35 106.5 mm to (42.3, 39.0), turned to 0 degrees
- moved U5 105.7 mm to (104.3, 40.8), turned to 0 degrees
- moved R1 104.0 mm to (188.1, 56.0), turned to 0 degrees
- moved R30 93.5 mm to (188.8, 78.0), turned to 0 degrees
- moved R3 92.9 mm to (190.2, 61.6), turned to 0 degrees
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Connections:
- J1 pad 2: VSS -> VEE
- J1 pad 3: Net-(J1-Pad3) -> DataCommand
- J2 pad 1: GND -> VCC
- J2 pad 2: Net-(J2-Pad2) -> GND
- J3 pad 2: Net-(J27-Pad3) -> Net-(J3-Pad2)
- J35 pad 19: Net-(J35-Pad19) -> MOSI
- J35 pad 2: Net-(J35-Pad2) -> VCC
- J35 pad 22: Net-(J35-Pad22) -> Reset
- J35 pad 23: Net-(J35-Pad23) -> SCLK
- J35 pad 26: Net-(J35-Pad26) -> ChipSelectEnable
- J35 pad 32: Net-(J35-Pad32) -> DataCommand
- J4 pad 2: Net-(J27-Pad4) -> Net-(J4-Pad2)
- R1 pad 1: Net-(Q1-Pad1) -> 1_TRS_MIDI_Tip
- R1 pad 2: Net-(R1-Pad2) -> Net-(J24-Pad2)
- R10 pad 1: Net-(Q10-Pad1) -> Net-(R10-Pad1)
- R10 pad 2: Net-(R10-Pad2) -> VCC
- R11 pad 1: Net-(Q11-Pad1) -> FootSw2
- R12 pad 1: Net-(Q12-Pad1) -> Net-(R11-Pad2)
- R12 pad 2: Net-(R12-Pad2) -> VCC
- R13 pad 1: Net-(Q13-Pad1) -> FootSw3
- R14 pad 1: Net-(Q14-Pad1) -> Net-(R13-Pad2)
- R14 pad 2: Net-(R14-Pad2) -> VCC
- R16 pad 1: Net-(J27-Pad5) -> 2_MIDI_Pin5
- R18 pad 1: Net-(J27-Pad6) -> 1_MIDI_Pin5
- R19 pad 1: MIDI_Rx -> FootSw4
- R19 pad 2: VCC -> Net-(R19-Pad2)
- R2 pad 1: Net-(Q2-Pad1) -> VCC
- R2 pad 2: Net-(R2-Pad2) -> Net-(J24-Pad3)
- R20 pad 1: Net-(D15-Pad2) -> Net-(R19-Pad2)
- R20 pad 2: Net-(J21-Pad5) -> VCC
- R3 pad 1: Net-(Q3-Pad1) -> 2_TRS_MIDI_Tip
- R3 pad 2: Net-(R3-Pad2) -> Net-(J25-Pad2)
- R30 pad 1: Net-(Q15-Pad1) -> VCC
- R4 pad 1: Net-(Q4-Pad1) -> VCC
- R4 pad 2: Net-(R4-Pad2) -> Net-(J25-Pad3)
- R5 pad 1: Net-(Q5-Pad1) -> 3_TRS_MIDI_Tip
- R5 pad 2: Net-(R4-Pad2) -> Net-(J3-Pad2)
- R6 pad 1: Net-(Q6-Pad1) -> VCC
- R6 pad 2: Net-(R6-Pad2) -> Net-(J3-Pad3)
- R7 pad 1: Net-(Q7-Pad1) -> 4_TRS_MIDI_Tip
- R7 pad 2: Net-(R6-Pad2) -> Net-(J4-Pad2)
- R8 pad 1: Net-(Q8-Pad1) -> VCC
- R8 pad 2: Net-(R8-Pad2) -> Net-(J4-Pad3)
- R9 pad 1: Net-(Q9-Pad1) -> FootSw1
- R9 pad 2: Net-(R9-Pad2) -> Net-(R10-Pad1)
- U10 pad 15: MIDI_Rx -> Net-(U10-Pad15)
- U2 pad 1: FootSw10 -> Net-(U2-Pad1)
- U2 pad 20: FootSw4 -> Net-(U2-Pad20)
- U2 pad 21: FootSw5 -> Net-(U2-Pad21)
- U2 pad 25: FootSw6 -> FootSw4
- U2 pad 26: FootSw7 -> Net-(U2-Pad26)
- U2 pad 27: FootSw8 -> FootSw5
- U2 pad 28: FootSw9 -> Net-(U2-Pad28)
- U5 pad 10: Net-(U5-Pad10) -> 2_TRS_MIDI_Tip
- U5 pad 11: Net-(U5-Pad11) -> MIDI_Tx
- U5 pad 12: Net-(U5-Pad12) -> 3_TRS_MIDI_Tip
- U5 pad 14: Net-(U5-Pad14) -> MIDI_Tx
- U5 pad 15: Net-(U5-Pad15) -> 4_TRS_MIDI_Tip
- U5 pad 2: 2_MIDI_Pin5 -> 1_MIDI_Pin5
- U5 pad 4: 1_MIDI_Pin5 -> 2_MIDI_Pin5
- U5 pad 6: Net-(U5-Pad6) -> 1_TRS_MIDI_Tip
- U5 pad 7: Net-(U5-Pad7) -> MIDI_Tx
- U5 pad 9: Net-(U5-Pad9) -> MIDI_Tx
Routing:
- net VCC: track 1120.4 -> 0.00 mm, vias 59 -> 0
- net Net-(J35-Pad3): track 395.9 -> 0.00 mm, vias 12 -> 0
- net Net-(J35-Pad5): track 345.7 -> 0.00 mm, vias 19 -> 0
- net Net-(C15-Pad2): track 232.8 -> 0.00 mm, vias 2 -> 0
- net Net-(C18-Pad2): track 164.3 -> 0.00 mm, vias 3 -> 0
- net Vol_In: track 163.1 -> 0.00 mm, vias 1 -> 0
- net MIDI_Tx: track 158.5 -> 0.00 mm, vias 12 -> 0
- net Net-(D2-Pad2): track 152.3 -> 0.00 mm, vias 7 -> 0
- net Net-(D22-Pad2): track 137.4 -> 0.00 mm, vias 6 -> 0
- net Net-(D17-Pad2): track 136.3 -> 0.00 mm, vias 4 -> 0
- net VSS: track 133.0 -> 0.00 mm, vias 6 -> 0
- net Net-(D7-Pad2): track 129.1 -> 0.00 mm, vias 4 -> 0
- net VEE: track 128.2 -> 0.00 mm, vias 6 -> 0
- net Tap4: track 127.8 -> 0.00 mm, vias 12 -> 0
- net Net-(D5-Pad2): track 127.7 -> 0.00 mm, vias 6 -> 0
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- removed copper zone on B.Cu, net GND
- removed copper zone on F.Cu, net GND
Other:
- board outline removed

Commit message: pcb almost done
Parts:
- moved J2 193.3 mm to (226.3, 51.3)
- moved J35 177.9 mm to (218.7, 62.2)
- moved J3 168.0 mm to (175.1, 46.1), turned to 90 degrees
- moved J1 167.5 mm to (200.3, 72.1), turned to 270 degrees
- moved R9 162.2 mm to (40.0, 147.5)
- moved J25 155.7 mm to (123.8, 45.5), turned to 90 degrees
- moved R10 151.7 mm to (39.6, 153.0), turned to 180 degrees
- moved R17 150.7 mm to (40.5, 58.1), turned to 270 degrees
- moved SW5 141.6 mm to (211.9, 50.9)
- moved C1 140.1 mm to (39.9, 141.2)
- moved R19 137.8 mm to (47.0, 86.2)
- moved J24 137.0 mm to (150.9, 46.2), turned to 90 degrees
- moved SW3 135.1 mm to (228.2, 141.3)
- moved R18 132.4 mm to (50.4, 58.3), turned to 90 degrees
- moved SW1 124.0 mm to (48.5, 142.6)
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Routing:
- net VCC: track 0.00 -> 713.8 mm, vias 0 -> 19
- net Net-(J35-Pad3): track 0.00 -> 202.1 mm, vias 0 -> 8
- net Net-(J35-Pad5): track 0.00 -> 198.9 mm, vias 0 -> 4
- net RotEncB: track 0.00 -> 156.1 mm
- net Net-(J35-Pad7): track 0.00 -> 150.8 mm, vias 0 -> 6
- net Net-(J35-Pad11): track 0.00 -> 148.3 mm, vias 0 -> 8
- net FootSw5: track 0.00 -> 147.6 mm, vias 0 -> 2
- net FootSw3: track 0.00 -> 131.7 mm
- net RotEncA: track 0.00 -> 83.8 mm, vias 0 -> 2
- net FootSw1: track 0.00 -> 81.4 mm
- net RotEncPushBttn: track 0.00 -> 78.7 mm, vias 0 -> 4
- net FootSw4: track 0.00 -> 72.0 mm
- net 3_TRS_MIDI_Tip: track 0.00 -> 66.8 mm
- net 1_MIDI_Pin5: track 0.00 -> 61.7 mm, vias 0 -> 2
- net Net-(R26-Pad1): track 0.00 -> 57.4 mm, vias 0 -> 1
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- added copper zone on B.Cu, net GND
- added copper zone on F.Cu, net GND
Other:
- board outline added: 202.8 x 137.6 mm

Commit message: modify pcb
Parts:
- C1, C13, C14, C5, R1, R10, R15, R16, R17, R18, R2, R21, R22, R3, R4, R5, R6, R68, R69, R7, R73, R74, R8, R9, U2: moved to B.Cu
- moved J8 108.6 mm to (109.7, 123.9), turned to 90 degrees
- moved R17 91.1 mm to (104.7, 122.8)
- moved J41 85.2 mm to (164.5, 126.6), turned to 270 degrees
- moved U2 77.1 mm to (164.2, 99.1)
- moved C13 76.2 mm to (145.1, 117.2), turned to 180 degrees
- moved C14 76.2 mm to (145.1, 114.1), turned to 180 degrees
- moved R30 76.1 mm to (202.6, 91.6), turned to 270 degrees
- moved R28 75.5 mm to (199.9, 91.6), turned to 270 degrees
- moved C7 75.1 mm to (197.2, 91.6), turned to 270 degrees
- moved R18 74.6 mm to (104.7, 109.5), turned to 270 degrees
- moved J7 70.2 mm to (109.8, 98.1), turned to 90 degrees
- moved U10 69.5 mm to (158.4, 115.5), turned to 180 degrees
- moved R69 68.2 mm to (141.0, 107.5), turned to 180 degrees
- moved C1 67.5 mm to (106.8, 132.1), turned to 270 degrees
- moved R9 65.8 mm to (104.0, 132.1), turned to 270 degrees
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Routing:
- net VCC: track 713.8 -> 93.1 mm, vias 19 -> 0
- net Net-(J35-Pad3): track 202.1 -> 4.37 mm, vias 8 -> 0
- net Net-(J35-Pad5): track 198.9 -> 4.53 mm, vias 4 -> 0
- net RotEncB: track 156.1 -> 0.00 mm
- net Net-(J35-Pad7): track 150.8 -> 0.00 mm, vias 6 -> 0
- net Net-(J35-Pad11): track 148.3 -> 0.00 mm, vias 8 -> 0
- net FootSw5: track 147.6 -> 0.00 mm, vias 2 -> 0
- net FootSw3: track 131.7 -> 0.00 mm
- net RotEncA: track 83.8 -> 0.00 mm, vias 2 -> 0
- net FootSw1: track 81.4 -> 0.00 mm
- net RotEncPushBttn: track 78.7 -> 0.00 mm, vias 4 -> 0
- net FootSw4: track 72.0 -> 0.00 mm
- net Net-(R26-Pad1): track 57.4 -> 0.00 mm, vias 1 -> 0
- net Net-(R24-Pad1): track 55.4 -> 0.00 mm
- net Net-(R23-Pad1): track 50.5 -> 0.00 mm
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Other:
- board size 202.8 x 137.6 mm -> 127 x 88.9 mm

Commit message: update pcb
Parts:
- moved J35 52.2 mm to (216.8, 68.5), turned to 0 degrees
- moved SW5 8.19 mm to (209.4, 58.9)
- moved C5 7.88 mm to (201.4, 59.0)
- moved R21 7.86 mm to (201.4, 61.7)
- moved R22 7.86 mm to (201.3, 64.6)
- moved J2 5.00 mm to (202.8, 70.7)
Routing:
- net VCC: track 93.1 -> 512.2 mm, vias 0 -> 19
- net FootSw1: track 0.00 -> 122.7 mm, vias 0 -> 2
- net FootSw4: track 0.00 -> 93.1 mm, vias 0 -> 3
- net Net-(J35-Pad5): track 4.53 -> 92.3 mm, vias 0 -> 6
- net Net-(J35-Pad3): track 4.37 -> 91.2 mm, vias 0 -> 6
- net FootSw5: track 0.00 -> 86.8 mm, vias 0 -> 4
- net FootSw3: track 0.00 -> 67.3 mm, vias 0 -> 3
- net Net-(J35-Pad11): track 0.00 -> 66.0 mm, vias 0 -> 4
- net RotEncA: track 0.00 -> 60.0 mm, vias 0 -> 7
- net Net-(J35-Pad7): track 0.00 -> 58.8 mm, vias 0 -> 3
- net RotEncPushBttn: track 0.00 -> 58.6 mm, vias 0 -> 4
- net FootSw2: track 0.00 -> 53.5 mm, vias 0 -> 3
- net Net-(J41-Pad1): track 0.00 -> 46.1 mm, vias 0 -> 1
- net Net-(R23-Pad1): track 0.00 -> 33.0 mm
- net Net-(R24-Pad1): track 0.00 -> 33.0 mm
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
Commit message: board finished. need fab files
Parts:
- J1: footprint Pin_Headers:Pin_Header_Straight_1x07_Pitch1.00mm -> Pin_Headers:Pin_Header_Straight_1x07_Pitch1.27mm
- moved J1 1.20 mm to (204.0, 102.0)
Routing:
- net Reset: track 26.2 -> 26.8 mm
- net (no net): vias 0 -> 327

Commit message: sent off board to be printed
Parts:
- moved C5 2.51 mm to (203.6, 57.8)
- moved R21 2.51 mm to (203.6, 60.5)
- moved R22 2.51 mm to (203.5, 63.4)
- moved SW5 1.90 mm to (211.3, 58.8)
Routing:
- net VCC: track 512.2 -> 514.3 mm
- net FootSw5: track 86.8 -> 88.5 mm
- net GND: vias 40 -> 439
- net (no net): vias 327 -> 0

Commit message: modify pcb
1. move the SPI chip enable wire that controls the OLED from rpi CE1 to CE0
2. swap r68 and r69 as they are in the wrong positions... opps
Parts:
- moved R69 9.25 mm to (137.6, 116.1), turned to 90 degrees
- moved R68 6.65 mm to (141.0, 109.6), turned to 0 degrees
Connections:
- J35 pad 24: Net-(J35-Pad24) -> ChipSelectEnable
- J35 pad 26: ChipSelectEnable -> Net-(J35-Pad26)
- R68 pad 1: VCC -> Net-(J41-Pad1)
- R69 pad 1: Net-(C14-Pad2) -> VCC
- R69 pad 2: Net-(J41-Pad1) -> Net-(C14-Pad2)
Routing:
- net ChipSelectEnable: track 28.2 -> 30.4 mm
- net Net-(J41-Pad1): track 46.1 -> 48.2 mm
- net Net-(C14-Pad2): track 11.3 -> 10.6 mm
- net VCC: track 514.3 -> 514.8 mm
